File: kicad/pico_radar_speed_sign/pico_radar_speed_sign.kicad_pcb (KiCad board)
At the start: 2 copper layers, 68 x 79 mm, 27 parts, among them J1 Conn_02x08_Odd_Even, J2 Conn_02x08_Odd_Even, J3 Conn_01x02, J4 Conn_01x03_Pin, J5 Conn_01x04, U1 Pico_H, U2 74HC595, U3 74HC595, U5 LM2596S-ADJ

Commit message: Make Pico controller Rev A
Parts:
- added C5: DNP, Capacitor_SMD:C_0805_2012Metric, F.Cu at (70.5, 69.0)
- added J6: 2.00mm JST-PH 01x03, Connector_JST:JST_PH_B3B-PH-K_1x03_P2.00mm_Vertical, F.Cu at (32.4, 133.5)
- J1, J2: value Conn_02x08_Odd_Even -> 0.1" Pin Header 02x08
- J4: value Conn_01x03_Pin -> 0.1" Pin Header 01x03
- moved R4 97.0 mm to (68.5, 69.0)
- moved H3 96.6 mm to (94.0, 135.0)
- moved H4 96.6 mm to (46.0, 135.0)
- moved C1 96.2 mm to (54.5, 85.0)
- moved C2 96.2 mm to (54.5, 101.5)
- moved C3 96.2 mm to (62.7, 78.8)
- moved C4 96.2 mm to (80.7, 69.5)
- moved D1 96.2 mm to (53.0, 78.0)
- moved GRAPHIC1 96.2 mm to (94.0, 127.5)
- moved H1 96.2 mm to (46.0, 64.0)
- moved H2 96.2 mm to (94.0, 64.0)
- moved J1 96.2 mm to (37.0, 122.0)
- moved J2 96.2 mm to (37.0, 97.8)
- moved J3 96.2 mm to (36.0, 66.9)
- moved J4 96.2 mm to (34.5, 134.1)
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Connections:
- J4 pad 1: /DOPPLER_RADAR_IN -> GND
- J4 pad 3: GND -> /DOPPLER_RADAR_IN
- U1 pad 1: /DOPPLER_RADAR_IN -> unconnected-(U1-GPIO0-Pad1)
- U1 pad 34: unconnected-(U1-GPIO28_ADC2-Pad34) -> /DOPPLER_RADAR_IN
Routing:
- net /DOPPLER_RADAR_IN: track 54.6 -> 39.1 mm
- net +5V: track 167.9 -> 171.4 mm
- net Net-(U5-FB): track 7.42 -> 8.17 mm
- net GND: vias 18 -> 17
Other:
- board text added: "2"
- board text added: "BACK"
- board text added: "FRONT"
- board text added: "NOTES 1. FABRICATE PCB IN ACCORDANCE WITH THE CURRENT REVISION OF IPC-6012, CLASS 2. 2. PCBA REVISION MUST BE MARKED WITH INDELIBLE INK ON THE BACK OF THE BOARD AT THE LOCATION SPECIFIED BY NOTE (2)."
- board text added: "Pico Radar Speed Sign Controller pantsforbirds.com"
- board text removed: "Pico Radar Speed Sign Control Board pantsforbirds.com"
