File: kicad/hb100_amplifier/hb100_amplifier.kicad_pcb (KiCad board)
At the start: 2 copper layers, 60 x 55.4 mm, 29 parts, among them J1 01x02 2.54mm Pin Socket, J2 01x02 2.54mm Pin Socket, J3 01x02 2.54mm Pin Socket, J4 01x02 2.54mm Pin Socket, J5 01x03 2.54mm Pin Header, U1 LM358, U2 AZ1117-3.3

Commit message: Add CPP firmware folder
Parts:
- R10: footprint Resistor_SMD:R_0402_1005Metric -> Resistor_SMD:R_0603_1608Metric
- moved R10 0.50 mm to (93.5, 43.0)

Commit message: Production files for extended range horn
Parts:
- U1: value LM358 -> LMV358; footprint Custom_Package_SO:SOP-8_3.76x4.96mm_P1.27mm -> Package_SO:SOIC-8_3.9x4.9mm_P1.27mm
- U2: value AZ1117-3.3 -> LM1117IMPX-3.3
- moved J2 2.54 mm to (67.5, 64.2)
