File: kicad/hb100_amplifier/hb100_amplifier.kicad_sch (KiCad schematic)
At the start: 29 parts, among them J1 01x02 2.54mm Pin Socket, J2 01x02 2.54mm Pin Socket, J3 01x02 2.54mm Pin Socket, J4 01x02 2.54mm Pin Socket, J5 01x03 2.54mm Pin Header, U1 LM358, U2 AZ1117-3.3

Commit message: Add CPP firmware folder
Parts:
- R8: footprint Resistor_SMD:R_0402_1005Metric -> Resistor_SMD:R_0603_1608Metric
Changed lines of the file:
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@@
       (effects (font (size 1.27 1.27)) (justify left))
     )
-    (property "Footprint" "Resistor_SMD:R_0402_1005Metric" (at 136.906 56.134 90)
+    (property "Footprint" "Resistor_SMD:R_0603_1608Metric" (at 136.906 56.134 90)
       (effects (font (size 1.27 1.27)) hide)
     )

Commit message: Production files for extended range horn
Parts:
- C1: LCSC PN (none) -> C1591; MPN (none) -> CL10B104KB8NNNC; Standard Cost (none) -> 0.01
- C11, C6, C8: LCSC PN (none) -> C1779; MPN (none) -> CL21A475KAQNNNE; Standard Cost (none) -> 0.02
- C2, C3, C4, C7: LCSC PN (none) -> C95841; MPN (none) -> CL21B106KOQNNNE; Standard Cost (none) -> 0.02
- C5, C9: LCSC PN (none) -> C16033; MPN (none) -> CL10B222KB8NNNC; Standard Cost (none) -> 0.01
- D1: LCSC PN (none) -> C963381; MPN (none) -> 1N5819W; Standard Cost (none) -> 0.05
- D3: LCSC PN (none) -> C510027
- J1, J2, J3, J4: LCSC PN (none) -> C49661; MPN (none) -> C49661
- J5: LCSC PN (none) -> C19190476; MPN (none) -> P125-1103A0BR138A1
- R1, R7: LCSC PN (none) -> C105578; MPN (none) -> RC0603FR-071ML; Standard Cost (none) -> 0.01
- R2: LCSC PN (none) -> C98220; MPN (none) -> RC0603FR-0710KL; Standard Cost (none) -> 0.01
- R3, R4: LCSC PN (none) -> C14675; MPN (none) -> RC0603FR-07100KL; Standard Cost (none) -> 0.01
- R5: LCSC PN (none) -> C114618; MPN (none) -> RC0603FR-07330KL; Standard Cost (none) -> 0.01
- R6: LCSC PN (none) -> C114637; MPN (none) -> RC0603FR-078K2L; Standard Cost (none) -> 0.01
- R8: LCSC PN (none) -> C227756; MPN RC0402FR-07287RL -> AC0603FR-07287RL
- R8: LCSC PN (none) -> C95177; MPN (none) -> RC0603JR-070RL; Standard Cost (none) -> 0.01
- R9: LCSC PN (none) -> C114659; MPN (none) -> RC0603FR-0712KL; Standard Cost (none) -> 0.01
- U1: value LM358 -> LMV358; footprint Custom_Package_SO:SOP-8_3.76x4.96mm_P1.27mm -> Package_SO:SOIC-8_3.9x4.9mm_P1.27mm; LCSC PN (none) -> C63813; MPN (none) -> LMV358IDR; Standard Cost (none) -> 0.10
- U2: value AZ1117-3.3 -> LM1117IMPX-3.3; LCSC PN (none) -> C23984; MPN (none) -> LM1117IMPX-3.3/NOPB; Standard Cost (none) -> 0.21
Other:
- company: (none) -> pantsforbirds.com
- title: (none) -> HB100 Amplifier
