File: kicad/hb100_horn_horizontal_wall/hb100_horn_horizontal_wall.kicad_pcb (KiCad board)
At the start: 2 copper layers, 75 x 60 mm, 0 parts

Commit message: Production files for extended range horn
Other:
- outline, holes or cut-outs redrawn
